File: pcbs/left/left-routed.kicad_pcb (KiCad board)
At the start: 2 copper layers, 111.6 x 82.4 mm, 47 parts, among them J1 Conn_01x12_Socket

Commit message: fix offset etc
Parts:
- added _1: VIA-0.6mm, VIA-0.6mm, F.Cu at (157.4, -128.1)
- added _2: VIA-0.6mm, VIA-0.6mm, F.Cu at (157.4, -125.5)
- added _3: VIA-0.6mm, VIA-0.6mm, F.Cu at (158.9, -128.1)
- added _4: VIA-0.6mm, VIA-0.6mm, F.Cu at (158.9, -125.5)
- added _5: VIA-0.6mm, VIA-0.6mm, F.Cu at (160.4, -128.1)
- added _6: VIA-0.6mm, VIA-0.6mm, F.Cu at (160.4, -125.5)
Routing:
- net R1: track 189.0 -> 195.5 mm
- net R2: track 186.9 -> 192.7 mm
- net C6: track 90.8 -> 94.8 mm, vias 1 -> 0
- net C5: track 171.6 -> 175.3 mm, vias 1 -> 0
- net GND: track 0.00 -> 3.70 mm, vias 0 -> 4
- net R4: track 114.2 -> 117.8 mm
- net C3: track 213.7 -> 217.2 mm, vias 1 -> 0
- net R3: track 214.4 -> 213.2 mm
- net C4: track 65.4 -> 66.1 mm, vias 1 -> 0
- net C1: track 115.2 -> 115.7 mm, vias 1 -> 0
- net C2: track 107.1 -> 107.2 mm, vias 1 -> 0
- added copper zone on B.Cu, net GND
- added copper zone on F.Cu, net GND
