File: pcbs/daughterboard/daughterboard/daughterboard.kicad_pcb (KiCad board)
At the start: 2 copper layers, 45 x 19.7 mm, 6 parts, among them J1 FFC2B28-12-G, J2 S2B-ZRLFSN, SW1 SW_Push

Commit message: final tweaks to pcbs before production
Parts:
- removed G***: LOGO, art:old_badger
- added REF**: baby_badger, art:baby_badger, B.Cu at (44.5, 42.5)
