File: pcbs/mainboard/mainboard.kicad_pcb (KiCad board)
At the start: 2 copper layers, 111.6 x 82.4 mm, 59 parts

Commit message: final tweaks to pcbs before production
Parts:
- added REF**: the46, art:the46, F.Cu at (174.0, 88.5)
- added REF**: righthand, art:righthand, F.Cu at (143.0, 105.2)
- added REF**: lefthand, art:lefthand, F.Cu at (137.8, 108.4)
- added REF**: the46, art:the46, B.Cu at (174.0, 89.5)
- added REF**: madeby, art:madeby, B.Cu at (109.2, 127.5)
- added REF**: old_badger_small, art:old_badger_small, B.Cu at (104.5, 123.5)
- moved _1 7.28 mm to (136.0, 85.0)
- moved _2 7.28 mm to (137.0, 85.0)
- moved _3 7.28 mm to (138.0, 85.0)
- moved _4 7.28 mm to (139.0, 85.0)
- moved _5 7.28 mm to (140.0, 85.0)
- moved _6 7.28 mm to (141.0, 85.0)
- moved _10 3.00 mm to (140.0, 78.0)
- moved _7 3.00 mm to (137.0, 78.0)
- moved _8 3.00 mm to (138.0, 78.0)
- moved _9 3.00 mm to (139.0, 78.0)
- moved D1 2.00 mm to (94.0, 90.8)
- moved D10 2.00 mm to (148.0, 129.0)
- moved D11 2.00 mm to (148.0, 112.0)
- moved D12 2.00 mm to (148.0, 95.0)
- moved D13 2.00 mm to (148.0, 78.0)
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Routing:
- net C3: track 79.5 -> 95.7 mm
- net R4: track 112.4 -> 120.8 mm
- net GND: track 0.00 -> 5.97 mm, vias 3 -> 6
- net R1: track 228.2 -> 223.6 mm
- net C2: track 116.2 -> 118.7 mm
- net R2: track 216.9 -> 214.7 mm
- net inner_thumb: track 19.0 -> 16.9 mm
- net ring_top: track 17.3 -> 15.3 mm
- net ring_thumb: track 17.3 -> 15.3 mm
- net ring_middle: track 17.3 -> 15.3 mm
- net ring_bottom: track 17.3 -> 15.3 mm
- net pinky_top: track 17.3 -> 15.3 mm
- net pinky_thumb: track 17.3 -> 15.3 mm
- net pinky_middle: track 17.3 -> 15.3 mm
- net pinky_bottom: track 17.3 -> 15.3 mm
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